Commit message: fix(MS-2): URDF 자체 검토 5건 수정 — 오도메트리 정확도·컨트롤러 안정성 개선
- wheel_separation 0.46→0.47 (정확한 계산값, SLAM 정밀도 영향)
- gazebo.launch.py 컨트롤러 로딩 레이스컨디션 수정 (spawn→JSB→DDC 이벤트 체이닝)
- CMakeLists.txt 미존재 meshes 디렉토리 참조 제거
- 센서 5종에 Gazebo material 태그 추가 (올바른 색상 렌더링)
- 센서 플랫폼 치수 하드코딩→dimensions.xacro 프로퍼티 통합

Co-Authored-By: Claude Opus 4.6 <noreply@anthropic.com>

File: ros2_ws/src/argos_description/urdf/platform/base.urdf.xacro (robot description, xacro)
@@ -69,5 +69,5 @@
     <visual>
       <geometry>
-        <box size="0.30 0.30 ${sensor_platform_height}"/>
+        <box size="${sensor_platform_length} ${sensor_platform_width} ${sensor_platform_height}"/>
       </geometry>
       <material name="argos_dark"/>
@@ -75,8 +75,8 @@
     <collision>
       <geometry>
-        <box size="0.30 0.30 ${sensor_platform_height}"/>
+        <box size="${sensor_platform_length} ${sensor_platform_width} ${sensor_platform_height}"/>
       </geometry>
     </collision>
-    <xacro:box_inertia m="0.5" x="0.30" y="0.30" z="${sensor_platform_height}"/>
+    <xacro:box_inertia m="0.5" x="${sensor_platform_length}" y="${sensor_platform_width}" z="${sensor_platform_height}"/>
   </link>
   <joint name="sensor_platform_joint" type="fixed">

File: ros2_ws/src/argos_description/urdf/platform/dimensions.xacro (robot description, xacro)
@@ -24,6 +24,8 @@
   <xacro:property name="wheel_x_offset"  value="0.20"/>
   <xacro:property name="wheel_y_offset"  value="${base_width / 2 + wheel_width / 2 + 0.01}"/>
-  <!-- ========== 센서 마운트 높이 ========== -->
-  <!-- base_link 위 센서 플랫폼 -->
+  <!-- ========== 센서 플랫폼 ========== -->
+  <!-- base_link 위 센서 마운트 상판 -->
+  <xacro:property name="sensor_platform_length" value="0.30"/>
+  <xacro:property name="sensor_platform_width"  value="0.30"/>
   <xacro:property name="sensor_platform_height" value="0.05"/>
   <xacro:property name="sensor_platform_z"       value="${base_height / 2 + sensor_platform_height / 2}"/>

File: ros2_ws/src/argos_description/urdf/sensors/depth_camera.urdf.xacro (robot description, xacro)
@@ -37,4 +37,8 @@
     </joint>
     <gazebo reference="${camera_name}_link">
+      <material>
+        <ambient>0.7 0.7 0.7 1.0</ambient>
+        <diffuse>0.7 0.7 0.7 1.0</diffuse>
+      </material>
       <sensor name="${camera_name}" type="depth_camera">
         <always_on>true</always_on>

File: ros2_ws/src/argos_description/urdf/sensors/imu.urdf.xacro (robot description, xacro)
@@ -30,4 +30,8 @@
     </joint>
     <gazebo reference="imu_link">
+      <material>
+        <ambient>1.0 0.8 0.0 1.0</ambient>
+        <diffuse>1.0 0.8 0.0 1.0</diffuse>
+      </material>
       <sensor name="imu" type="imu">
         <always_on>true</always_on>

File: ros2_ws/src/argos_description/urdf/sensors/lidar.urdf.xacro (robot description, xacro)
@@ -31,4 +31,8 @@
     </joint>
     <gazebo reference="lidar_link">
+      <material>
+        <ambient>0.15 0.15 0.15 1.0</ambient>
+        <diffuse>0.15 0.15 0.15 1.0</diffuse>
+      </material>
       <sensor name="gpu_lidar" type="gpu_lidar">
         <always_on>true</always_on>

File: ros2_ws/src/argos_description/urdf/sensors/rgb_camera.urdf.xacro (robot description, xacro)
@@ -38,4 +38,8 @@
     </joint>
     <gazebo reference="${camera_name}_link">
+      <material>
+        <ambient>0.15 0.15 0.15 1.0</ambient>
+        <diffuse>0.15 0.15 0.15 1.0</diffuse>
+      </material>
       <sensor name="${camera_name}" type="camera">
         <always_on>true</always_on>

File: ros2_ws/src/argos_description/urdf/sensors/thermal_camera.urdf.xacro (robot description, xacro)
@@ -39,4 +39,8 @@
     </joint>
     <gazebo reference="${camera_name}_link">
+      <material>
+        <ambient>1.0 0.8 0.0 1.0</ambient>
+        <diffuse>1.0 0.8 0.0 1.0</diffuse>
+      </material>
       <sensor name="${camera_name}" type="thermal_camera">
         <always_on>true</always_on>
