Commit message: feat: v2.0 아키텍처 대폭 보완 — LifecycleNode 4노드 + DimOS 벤치마킹 4기능 + Nav2 안정화
주요 변경:
- LifecycleNode 전환: orchestrator, frontier_explorer, hotspot_detector, gas_sensor
- TF frame_prefix: 멀티로봇 TF 격리 (namespace remapping → frame_prefix)
- Nav2 DDC 체이닝: TimerAction → OnProcessExit(ddc_spawner) + 45s 대기
- DimOS 벤치마킹 4기능: SkillLibrary(393줄), MCP 서버(279줄), ReactiveStream(337줄), Rerun 브릿지(296줄)
- Kalman 시계열 강화: 142→380줄 (시간기반 추적, 화점-피해자 근접경고, 확산추세)
- launch_testing 통합 테스트 3개 (화재 대응, 멀티로봇 경합, 배터리 lifecycle)
- pytest-cov 설정, rosbridge TLS launch 인자, gz_bridge 헬스체크 스크립트
- 열화상 카메라 20Hz, slam_toolbox transform_timeout 2.0s
- 8중 센싱 체계, CI/CD, Dockerfile, 15명 전문가 리뷰 (83→89점)

테스트: 511 passed (WSL2), 491 passed (Windows)
빌드: colcon build 4패키지 성공
검증: Gazebo headless cmd_vel +6.35m 이동 확인

Co-Authored-By: Claude Opus 4.6 (1M context) <noreply@anthropic.com>

File: ros2_ws/src/argos_description/urdf/platform/dimensions.xacro (robot description, xacro)
@@ -11,14 +11,26 @@
 <robot xmlns:xacro="http://www.ros.org/wiki/xacro">
   <!-- ========== 섀시 ========== -->
+  <!-- HW 전문가 권고: 15kg→8kg (알루미늄 6061 프레임 기준, TurtleBot Waffle 스케일링) -->
+  <!-- 상세: docs/hardware-design-spec.md 질량 재검증 섹션 -->
   <xacro:property name="base_length"  value="0.60"/>
   <xacro:property name="base_width"   value="0.40"/>
   <xacro:property name="base_height"  value="0.15"/>
-  <xacro:property name="base_mass"    value="15.0"/>
+  <xacro:property name="base_mass"    value="8.0"/>
   <!-- 지면으로부터 섀시 바닥까지 간격 -->
   <xacro:property name="ground_clearance" value="0.05"/>
   <!-- ========== 바퀴 ========== -->
+  <!-- HW 전문가 권고: 1.0kg→0.5kg (소형 UGV 고무 바퀴 기준) -->
   <xacro:property name="wheel_radius"    value="0.10"/>
   <xacro:property name="wheel_width"     value="0.05"/>
-  <xacro:property name="wheel_mass"      value="1.0"/>
+  <xacro:property name="wheel_mass"      value="0.5"/>
+  <!-- ========== 배터리 (HW 전문가 권고: 신규) ========== -->
+  <!-- 4S LiPo 14.8V 10000mAh, ~800g -->
+  <xacro:property name="battery_mass"    value="0.8"/>
+  <xacro:property name="battery_length"  value="0.15"/>
+  <xacro:property name="battery_width"   value="0.08"/>
+  <xacro:property name="battery_height"  value="0.05"/>
+  <!-- 배터리 위치: 섀시 후방 중앙 (CoG 균형) -->
+  <xacro:property name="battery_x"       value="-0.15"/>
+  <xacro:property name="battery_z"       value="0.0"/>
   <!-- 바퀴 위치 (섀시 중심 기준) -->
   <xacro:property name="wheel_x_offset"  value="0.20"/>

File: ros2_ws/src/argos_description/urdf/sensors/rgb_camera.urdf.xacro (robot description, xacro)
@@ -48,5 +48,5 @@
         <gz_frame_id>${camera_name}_optical_link</gz_frame_id>
         <camera>
-          <horizontal_fov>1.3962634</horizontal_fov>
+          <horizontal_fov>1.7453293</horizontal_fov>  <!-- 100° (HW 전문가 권고: 80°→100°) -->
           <image>
             <width>640</width>

File: ros2_ws/src/argos_description/urdf/sensors/thermal_camera.urdf.xacro (robot description, xacro)
@@ -45,5 +45,6 @@
       <sensor name="${camera_name}" type="thermal_camera">
         <always_on>true</always_on>
-        <update_rate>10</update_rate>
+        <!-- HW 전문가 권고: 10→20Hz (화점 이동 추적 정밀도 향상) -->
+        <update_rate>20</update_rate>
         <topic>${topic}</topic>
         <gz_frame_id>${camera_name}_optical_link</gz_frame_id>
@@ -51,6 +52,6 @@
           <horizontal_fov>0.6981317</horizontal_fov>
           <image>
-            <width>160</width>
-            <height>120</height>
+            <width>320</width>
+            <height>240</height>
             <format>L8</format>
           </image>
