Commit message: feat(MS-5): 멀티로봇 네임스페이스 분리 — N대 동시 스폰 지원
xacro namespace/topic_prefix 파라미터, controllers.yaml 와일드카드,
gz_ros2_control <ros><namespace> 태그, per-robot launch 그룹 구성.
단일 로봇(gazebo.launch.py) 하위호환 유지.

Co-Authored-By: Claude Opus 4.6 <noreply@anthropic.com>

File: ros2_ws/src/argos_description/urdf/argos_ugv.urdf.xacro (robot description, xacro)
@@ -11,7 +11,13 @@
 -->
 <robot name="argos_ugv" xmlns:xacro="http://www.ros.org/wiki/xacro">
-  <!-- ===== 시뮬레이션 모드 파라미터 ===== -->
+  <!-- ===== 파라미터 ===== -->
   <xacro:arg name="use_sim" default="true"/>
+  <xacro:arg name="namespace" default=""/>
+  <xacro:arg name="robot_name" default="argos_ugv"/>
   <xacro:property name="use_sim" value="$(arg use_sim)"/>
+  <xacro:property name="ns" value="$(arg namespace)"/>
+  <xacro:property name="robot_name" value="$(arg robot_name)"/>
+  <!-- 네임스페이스 접두사: 비어있으면 "" / 있으면 "/ns" -->
+  <xacro:property name="topic_prefix" value="${'/' + ns if ns != '' else ''}"/>
   <!-- ===== 1. Platform 계층 ===== -->
   <xacro:include filename="$(find argos_description)/urdf/platform/base.urdf.xacro"/>
@@ -29,5 +35,5 @@
     parent_link="sensor_platform_link"
     xyz="0 0 ${sensor_platform_height/2 + 0.02}"
-    topic="/scan"/>
+    topic="${topic_prefix}/scan"/>
   <!-- RGB 카메라: 전방 상단 -->
   <xacro:rgb_camera
@@ -35,5 +41,5 @@
     xyz="${camera_x} 0 ${camera_z}"
     camera_name="front_camera"
-    topic="/camera/image_raw"/>
+    topic="${topic_prefix}/camera/image_raw"/>
   <!-- 깊이 카메라: RGB 카메라 옆 (RealSense 위치) -->
   <xacro:depth_camera
@@ -41,10 +47,10 @@
     xyz="${camera_x} 0.04 ${camera_z}"
     camera_name="depth_camera"
-    topic="/depth_camera"/>
+    topic="${topic_prefix}/depth_camera"/>
   <!-- IMU: 섀시 중심 -->
   <xacro:imu_sensor
     parent_link="base_link"
     xyz="0 0 0"
-    topic="/imu/data"/>
+    topic="${topic_prefix}/imu/data"/>
   <!-- 열화상 카메라: 전방 하단 (화점 감지용) -->
   <xacro:thermal_camera
@@ -52,6 +58,6 @@
     xyz="${camera_x} 0 ${-base_height/2 + 0.05}"
     camera_name="thermal_camera"
-    topic="/thermal/image_raw"/>
+    topic="${topic_prefix}/thermal/image_raw"/>
   <!-- ===== ros2_control 인스턴스화 ===== -->
-  <xacro:argos_ros2_control use_sim="${use_sim}"/>
+  <xacro:argos_ros2_control use_sim="${use_sim}" namespace="${ns}"/>
 </robot>

File: ros2_ws/src/argos_description/urdf/control/ros2_control.urdf.xacro (robot description, xacro)
@@ -7,5 +7,5 @@
 -->
 <robot xmlns:xacro="http://www.ros.org/wiki/xacro">
-  <xacro:macro name="argos_ros2_control" params="use_sim:='true'">
+  <xacro:macro name="argos_ros2_control" params="use_sim:='true' namespace:=''">
     <ros2_control name="ArgosSystem" type="system">
       <hardware>
@@ -60,4 +60,7 @@
         <plugin filename="gz_ros2_control-system" name="gz_ros2_control::GazeboSimROS2ControlPlugin">
           <parameters>$(find argos_description)/config/controllers.yaml</parameters>
+          <ros>
+            <namespace>${namespace}</namespace>
+          </ros>
         </plugin>
       </gazebo>
